Commit message: lifecycle slam_toolbox, URDF fixes, robot image OpenSSL
slam_toolbox (Humble/Jazzy lifecycle node)
- After a delay, run configure + activate so /scan and /map work in mapping,
  localization, and online_async launches (override slam_activate_delay).
- Tune mapper_params_online_async: faster map updates and scan matching,
  lower minimum travel/heading; document LD08 beam-count vs Karto (#426).

TurtleBot3 description (burger + waffle)
- Move Z pi from scan_joint to base_joint so LDS-02 + meshes line up in RViz.
- Flip wheel joint axes to negative Z so joint_state signs match physical spin.
- rfid_base_link rpy uses full pi constant.

Robot Docker / merge
- Set OPENSSL_ROOT_DIR and PKG_CONFIG_PATH per arch so Fast-DDS finds OpenSSL
  under QEMU arm64 builds; install libssl3.
- merge_src.sh: skip build/install/log so mistaken colcon output under src is
  not copied into the image context.

Dev UX
- AGENTS.md + cursor rules: LiDAR TF note, docker context hints.
- scripts/robot README: large robot_description / dump helpers.
- scripts/pc: build_ros, docker_build_robot, run_rviz_robot, README tweaks.
- rviz_configs/rviz_1.rviz: display updates.

Teleop
- Optional TELEOP_INVERT_LINEAR / TELEOP_INVERT_ANGULAR for sim vs real
  diff-drive sign conventions.

Untracked (add if part of this change): .dockerignore, scripts/robot/
dump_robot_description.sh, get_robot_description_param.py, scripts/pc/
teleop_keyboard.sh, ros2_ws/src/turtlebot3_teleop/

File: turtlebot3/turtlebot3_description/urdf/turtlebot3_burger.urdf (robot description, URDF)
Before this commit: robot turtlebot3_burger, 9 links, 8 joints
Joints:
- joint base_joint: origin xyz=0.0 0.0 0.010 rpy=0 0 0 -> xyz=0.0 0.0 0.010 rpy=0 0 3.141592653589793
- joint wheel_left_joint: axis 0 0 1 -> 0 0 -1
- joint wheel_right_joint: axis 0 0 1 -> 0 0 -1

File: turtlebot3/turtlebot3_description/urdf/turtlebot3_waffle.urdf (robot description, URDF)
Before this commit: robot turtlebot3_waffle, 13 links, 12 joints
Joints:
- joint base_joint: origin xyz=0 0 0.010 rpy=0 0 0 -> xyz=0 0 0.010 rpy=0 0 3.141592653589793
- joint wheel_left_joint: axis 0 0 1 -> 0 0 -1
- joint wheel_right_joint: axis 0 0 1 -> 0 0 -1

File: turtlebot3/turtlebot3_description/urdf/turtlebot3_waffle_pi.urdf (robot description, URDF)
Before this commit: robot turtlebot3_waffle_pi, 11 links, 10 joints
Joints:
- joint base_joint: origin xyz=0 0 0.010 rpy=0 0 0 -> xyz=0 0 0.010 rpy=0 0 3.141592653589793
- joint wheel_left_joint: axis 0 0 1 -> 0 0 -1
- joint wheel_right_joint: axis 0 0 1 -> 0 0 -1
